File: RS485-CANBUS-WeMos.brd (EAGLE design)
At the start: 25.4 x 33 mm, 27 parts, among them J1 1X2-3.5MM, J2 1X2-3.5MM, J3 1X2-3.5MM, Q2 BC817, U1 MCP2551, U2 SP3485, U3 AOZ1282

Commit message: New revision
Parts:
- removed D1: SS14, adafruit:SOD-323F
- removed Q2: BC817, transistor-npn:SOT23-BEC
- removed R2: 10k, SparkFun:0805
- removed R8: 51k, SparkFun-Resistors:0805
- removed R9: 10k, SparkFun-Resistors:0805
- C1, C2, C4, C5: device SparkFun-Capacitors:0805 -> SparkFun:0805
- C3: value 10uF -> 10u; device SparkFun-Capacitors:1206 -> SparkFun:1210
- L1: value 22uH -> 4.7μH; device TaaraLabs:1210 -> SparkFun-Coils:INDUCTOR_4X4MM
- R3: value 1k -> 120; device SparkFun-Resistors:0805 -> SparkFun:0805
- R4: device SparkFun-Resistors:0805 -> SparkFun:0805
- R5: value 1k -> 10k; device SparkFun-Resistors:0805 -> SparkFun:0805
- R6: value 220 -> 120; device SparkFun-Resistors:0805 -> SparkFun:0805
- U1: value MCP2551 -> SN65HVD232
- U2: value SP3485 -> THVD1406
- U3: value AOZ1282 -> AP63203; device TaaraLabs:SOT23-6 -> SparkFun-IC-Power:SOT23-6
- moved R3 11.1 mm to (9.53, 21.6), turned to 180 degrees
- moved L1 10.3 mm to (17.8, 12.1), turned to 90 degrees
- moved C3 10.3 mm to (7.62, 12.1)
- moved C4 8.84 mm to (17.8, 15.9)
- moved R7 8.84 mm to (7.62, 15.9), turned to 0 degrees
- moved J1 6.98 mm to (5.71, 3.81)
- moved J2 6.98 mm to (12.7, 3.81)
- moved C1 6.75 mm to (5.08, 26.7)
- moved R1 2.54 mm to (5.08, 24.1)
- moved R4 2.54 mm to (20.3, 24.1), turned to 180 degrees
- moved U3 1.91 mm to (12.7, 14.6), turned to 270 degrees
- moved U$2 0.64 mm to (12.7, 17.1)
- turned R6 to 0 degrees
- turned U1 to 180 degrees
Connections:
- net N$1 renamed RS
- removed net 5V: C1.1, C2.1, C5.1, H2.8, L1.2, R4.1, R8.2, U1.3, U2.8
- removed net FB: R8.1, R9.2, U3.3
- removed net LX: C4.2, D1.C, L1.1, U3.6
- removed net N$2: R2.1, U1.4
- removed net N$3: R3.1, U2.1
- removed net N$4: Q2.C, R4.2, U2.2, U2.3
- removed net N$5: Q2.B, R5.2
- new net /SHDN: R5.1, U2.2, U2.3
- new net SW: C4.2, L1.P$1, U3.5
- net 12V: now also U3.3; no longer U3.5
- net 3.3V: now also C1.1, C2.1, C5.1, L1.P$2, R4.2, R5.2, U1.3, U2.8, U3.1
- net A: now also R6.1; no longer R6.2
- net B: now also R6.2; no longer R6.1
- net BST: now also U3.6; no longer U3.1
- net CANRXD: now also U1.4; no longer R2.2
- net EN: now also U3.2; no longer U3.4
- net GND: now also U3.4; no longer D1.A, Q2.E, R9.1, U2.4, U3.2
- net H: now also J1.1, R3.1; no longer J1.2
- net L: now also J1.2, R3.2; no longer J1.1
- net UARTRXD: now also H2.6, R4.1, U2.1; no longer H2.2, R3.2
- net UARTTXD: now also H2.5, U2.4; no longer H2.1, R5.1
Routing:
- net 3.3V: track 0.00 -> 89.3 mm
- net 5V: track 75.5 -> 0.00 mm
- net UARTTXD: track 2.91 -> 25.7 mm
- net UARTRXD: track 2.91 -> 22.7 mm
- net N$4: track 16.2 -> 0.00 mm
- net H: track 43.9 -> 28.8 mm
- net L: track 39.9 -> 25.2 mm
- net GND: track 22.8 -> 36.0 mm, vias 9 -> 7
- net CANTXD: track 11.3 -> 23.2 mm
- net CANRXD: track 7.40 -> 19.0 mm
- net N$2: track 11.3 -> 0.00 mm
- net /SHDN: track 0.00 -> 8.93 mm
- net SW: track 0.00 -> 8.26 mm
- net 12V: track 27.3 -> 20.0 mm
- net FB: track 6.52 -> 0.00 mm
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