File: RS485-CANBUS-WeMos.sch (EAGLE design)
At the start: 25 parts, among them J1 1X2-3.5MM, J2 1X2-3.5MM, J3 1X2-3.5MM, Q2 BC817, U1 MCP2551, U2 SP3485, U3 AOZ1282

Commit message: New revision
Parts:
- removed D1: SS14, adafruit:DIODESOD-323F
- removed Q2: BC817, transistor-npn:BC817-16SMD
- removed R2: 10k, SparkFun:RESISTOR0805-RES
- removed R8: 51k, SparkFun-Resistors:0.3OHM-0805-1/8W-1%
- removed R9: 10k, SparkFun-Resistors:0.3OHM-0805-1/8W-1%
- C1, C2, C4, C5: device SparkFun-Capacitors:1.0UF-0805-25V-10% -> SparkFun:CAP0805
- C3: value 10uF -> 10u; device SparkFun-Capacitors:1.0UF-1206-50V-10% -> SparkFun:CAP1210
- L1: value 22uH -> 4.7μH; device TaaraLabs:INDUCTOR1210 -> SparkFun-Coils:4.7μH_SHIELDED_INDUCTORNPIS_LS
- R3: value 1k -> 120; device SparkFun-Resistors:0.3OHM-0805-1/8W-1% -> SparkFun:RESISTOR0805-RES
- R4: device SparkFun-Resistors:0.3OHM-0805-1/8W-1% -> SparkFun:RESISTOR0805-RES
- R5: value 1k -> 10k; device SparkFun-Resistors:0.3OHM-0805-1/8W-1% -> SparkFun:RESISTOR0805-RES
- R6: value 220 -> 120; device SparkFun-Resistors:0.3OHM-0805-1/8W-1% -> SparkFun:RESISTOR0805-RES
- U1: value MCP2551 -> SN65HVD232
- U2: value SP3485 -> THVD1406
- U3: value AOZ1282 -> AP63203; device TaaraLabs:AOZ1282CI -> SparkFun-IC-Power:AP63203
Connections:
- net N$1 renamed RS
- removed net 5V: C1.1, C2.1, C5.1, H2.8, L1.2, R4.1, R8.2, U1.VDD, U2.VCC
- removed net FB: R8.1, R9.2, U3.FB
- removed net LX: C4.2, D1.C, L1.1, U3.LX
- removed net N$2: R2.1, U1.RXD
- removed net N$3: R3.1, U2.RO
- removed net N$4: Q2.C, R4.2, U2./RE, U2.DE
- removed net N$5: Q2.B, R5.2
- new net /SHDN: R5.1, U2./RE, U2.DE
- new net SW: C4.2, L1.1, U3.SW
- net 3.3V: now also C1.1, C2.1, C5.1, L1.2, R4.2, R5.2, U1.VDD, U2.VCC, U3.FB
- net A: now also R6.1; no longer R6.2
- net B: now also R6.2; no longer R6.1
- net CANRXD: now also U1.RXD; no longer R2.2
- net GND: no longer D1.A, Q2.E, R9.1, U2.DI
- net H: now also J1.1, R3.1; no longer J1.2
- net L: now also J1.2, R3.2; no longer J1.1
- net UARTRXD: now also H2.6, R4.1, U2.RO; no longer H2.2, R3.2
- net UARTTXD: now also H2.5, U2.DI; no longer H2.1, R5.1
Other:
- note added: "CAN+RS485+DCDC WeMos v1"
- note added: "v1.9 (2023-07-30)"
- note removed: "CAN+RS485 WeMos v1"
- note removed: "v1 (2023-06-04)"
- moved on the sheet: C1, C2, C4, C5, R3, R4, R5, R6, R7, U2
